Commit message: UPDATE:
modified xacro for rviz

File: src/TechControlInterface/description/urdf/create_link.xacro (robot description, xacro)
@@ -5,12 +5,12 @@
         xyz_offset
         rpy_offset
+        mass
         mesh_path">
     <link name="${link_name}">
-      <visual>
+      <inertial>
         <origin xyz="${xyz_offset}" rpy="${rpy_offset}"/>
-        <geometry>
-          <mesh filename="${mesh_path}/${link_name}.STL"/>
-        </geometry>
-      </visual>
+        <mass value="1"/>
+        <inertia ixx="1.0" ixy="0.0" ixz="0.0" iyy="1.0" iyz="0.0" izz="1.0"/>
+      </inertial>
       <collision>
         <origin xyz="0 0 0" rpy="0 0 0"/>
@@ -19,8 +19,17 @@
         </geometry>
       </collision>
-      <inertial>
-        <mass value="1"/>
-        <inertia ixx="1.0" ixy="0.0" ixz="0.0" iyy="1.0" iyz="0.0" izz="1.0"/>
-      </inertial>
+      <visual>
+        <origin
+          xyz="0 0 0"
+          rpy="0 0 0" />
+        <material
+          name="">
+          <color
+            rgba="1 1 1 1" />
+        </material>
+        <geometry>
+          <mesh filename="${mesh_path}/${link_name}.STL"/>
+        </geometry>
+      </visual>
     </link>
   </xacro:macro>

File: src/TechControlInterface/description/urdf/robot_description.urdf.xacro (robot description, xacro)
@@ -8,4 +8,5 @@
       xyz_offset="0.134546485528339 1.02602768939509 0.0276854546001787"
       rpy_offset="0 0 0"
+      mass="23.3444937848516"
       mesh_path="package://TechControlInterface/meshes"
   />
@@ -14,4 +15,5 @@
       xyz_offset="0.109505946566475 1.56830006166103 0.306532290779036"
       rpy_offset="0 0 0"
+      mass="8.67027571199243"
       mesh_path="package://TechControlInterface/meshes"
   />
@@ -20,4 +22,5 @@
       xyz_offset="0.0601483990121618 -0.443944828019226 1.73584633920143E-05"
       rpy_offset="0 0 0"
+      mass="0.647403062770475"
       mesh_path="package://TechControlInterface/meshes"
   />
@@ -26,4 +29,5 @@
       xyz_offset="-0.16447187278791 0.0126535013198428 0.1148075556278"
       rpy_offset="0 0 0"
+      mass="0.647403062770475"
       mesh_path="package://TechControlInterface/meshes"
   />
@@ -32,4 +36,5 @@
       xyz_offset="-0.0679648513950829 -0.0125948841535013 0.0597190016437489"
       rpy_offset="0 0 0"
+      mass="0.441881459418396"
       mesh_path="package://TechControlInterface/meshes"
   />
@@ -38,4 +43,5 @@
       xyz_offset="-2.79564493776974E-08 -0.00496995620296214 0.0493158936775911"
       rpy_offset="0 0 0"
+      mass="0.359995634810237"
       mesh_path="package://TechControlInterface/meshes"
   />
@@ -44,4 +50,5 @@
       xyz_offset="-0.0043261798092078 0.0995606848099331 0.196143761355562"
       rpy_offset="0 0 0"
+      mass="0.441881459418396"
       mesh_path="package://TechControlInterface/meshes"
   />
@@ -50,4 +57,5 @@
       xyz_offset="0.000386879822536601 -0.0239742458499962 0.247370540938741"
       rpy_offset="0 0 0"
+      mass="0.441881459418396"
       mesh_path="package://TechControlInterface/meshes"
   />
