Commit message: TMPSAVE: daily update

File: src/TechControlInterface/description/ros2_control/TechJoints.ros2_control.xacro (robot description, xacro)
@@ -10,6 +10,8 @@
         <command_interface name="position"/>
         <state_interface name="position"/>
+        <command_interface name="velocity"/>
+        <state_interface name="velocity"/>
       </joint>
-      <joint name="${prefix}joint3">
+      <!-- <joint name="${prefix}joint3">
         <command_interface name="position"/>
         <state_interface name="position"/>
@@ -22,5 +24,5 @@
         <command_interface name="position"/>
         <state_interface name="position"/>
-      </joint>
+      </joint> -->
     </ros2_control>
   </xacro:macro>

Commit message: MILESTONE: 4 Tech joint can be control by qt ui

File: src/TechControlInterface/description/ros2_control/TechJoints.ros2_control.xacro (robot description, xacro)
@@ -13,16 +13,22 @@
         <state_interface name="velocity"/>
       </joint>
-      <!-- <joint name="${prefix}joint3">
+      <joint name="${prefix}joint3">
         <command_interface name="position"/>
         <state_interface name="position"/>
+        <command_interface name="velocity"/>
+        <state_interface name="velocity"/>
       </joint>
       <joint name="${prefix}joint4">
         <command_interface name="position"/>
         <state_interface name="position"/>
+        <command_interface name="velocity"/>
+        <state_interface name="velocity"/>
       </joint>
         <joint name="${prefix}joint5">
         <command_interface name="position"/>
         <state_interface name="position"/>
-      </joint> -->
+        <command_interface name="velocity"/>
+        <state_interface name="velocity"/>
+      </joint>
     </ros2_control>
   </xacro:macro>

Commit message: UPDATE: different driver init together

File: src/TechControlInterface/description/ros2_control/TechJoints.ros2_control.xacro (robot description, xacro)
@@ -31,4 +31,10 @@
         <state_interface name="velocity"/>
       </joint>
+      <joint name="${prefix}joint6">
+        <command_interface name="position"/>
+        <state_interface name="position"/>
+        <command_interface name="velocity"/>
+        <state_interface name="velocity"/>
+      </joint>
     </ros2_control>
   </xacro:macro>

File: src/TechControlInterface/description/urdf/robot_description.urdf.xacro (robot description, xacro)
@@ -71,5 +71,7 @@
     <parent link="base_link"/>
     <child link="link0"/>
-    <origin xyz="0 0 0.061584" rpy="0 0 0"/>
+    <origin
+     xyz="0 -1 0.061584"
+     rpy="0 0 0"/>
     <axis xyz="0 -1 0"/>
     <limit effort="1000.0" lower="-1" upper="1" velocity="2.5"/>
@@ -89,5 +91,5 @@
     <origin
       xyz="0.149 -0.36401 0"
-      rpy="0 0 1.5708" />
+      rpy="1.680577537 0 1.5708" />
     <axis xyz="1 0 0"/>
     <limit effort="1000.0" lower="${-pi}" upper="${pi}" velocity="2.5"/>
@@ -98,5 +100,5 @@
     <origin
       xyz="-0.01 0.027384 0.2485"
-      rpy="0 0 0" />
+      rpy="-0.317649924 0 0" />
     <axis xyz="1 0 0"/>
     <limit effort="1000.0" lower="${-pi}" upper="${pi}" velocity="2.5"/>
@@ -116,5 +118,5 @@
     <origin
       xyz="0 -0.0735 0.0645"
-      rpy="1.5708 1.363 -3.1416" />
+      rpy="1.5708 0.187869814 -3.1416" />
     <axis xyz="0 0 -1"/>
     <limit effort="1000.0" lower="${-pi}" upper="${pi}" velocity="2.5"/>

Commit message: TMPSAVE: TODO: 1. find out relationship between hardware, controller and moveit2. Currently block out position controller. 2.move_config should use infomation in TechInterface pkg. 3. We need a cartesian path in ui.
TMPSAVE:
bug in judgement in swtiching mode in hw_if.

UPDATE:
1. moveit is available now!
2. Ban RobotUI temporarily cause the unit of velocity and position is defined up to encoder resolution.

File: src/TechControlInterface/description/ros2_control/TechJoints.ros2_control.xacro (robot description, xacro)
@@ -31,10 +31,10 @@
         <state_interface name="velocity"/>
       </joint>
-      <joint name="${prefix}joint6">
+      <!-- <joint name="${prefix}joint6">
         <command_interface name="position"/>
         <state_interface name="position"/>
         <command_interface name="velocity"/>
         <state_interface name="velocity"/>
-      </joint>
+      </joint> -->
     </ros2_control>
   </xacro:macro>

File: src/TechControlInterface/description/urdf/create_link.xacro (robot description, xacro)
@@ -9,5 +9,5 @@
     <link name="${link_name}">
       <inertial>
-        <origin xyz="${xyz_offset}" rpy="${rpy_offset}"/>
+        <origin xyz="0 0 0" rpy="0 0 0"/>
         <mass value="1"/>
         <inertia ixx="1.0" ixy="0.0" ixz="0.0" iyy="1.0" iyz="0.0" izz="1.0"/>
@@ -20,7 +20,5 @@
       </collision>
       <visual>
-        <origin
-          xyz="0 0 0"
-          rpy="0 0 0" />
+        <origin xyz="${xyz_offset}" rpy="${rpy_offset}"/>
         <material
           name="">

File: src/TechControlInterface/description/urdf/robot_description.urdf.xacro (robot description, xacro)
@@ -6,5 +6,5 @@
   <xacro:create_link
       link_name="base_link"
-      xyz_offset="0.134546485528339 1.02602768939509 0.0276854546001787"
+      xyz_offset="0 0 0"
       rpy_offset="0 0 0"
       mass="23.3444937848516"
@@ -13,5 +13,5 @@
   <xacro:create_link
       link_name="link0"
-      xyz_offset="0.109505946566475 1.56830006166103 0.306532290779036"
+      xyz_offset="0 0 0"
       rpy_offset="0 0 0"
       mass="8.67027571199243"
@@ -20,5 +20,5 @@
   <xacro:create_link
       link_name="link1"
-      xyz_offset="0.0601483990121618 -0.443944828019226 1.73584633920143E-05"
+      xyz_offset="0 0 0"
       rpy_offset="0 0 0"
       mass="0.647403062770475"
@@ -27,5 +27,5 @@
   <xacro:create_link
       link_name="link2"
-      xyz_offset="-0.16447187278791 0.0126535013198428 0.1148075556278"
+      xyz_offset="0 0 0"
       rpy_offset="0 0 0"
       mass="0.647403062770475"
@@ -34,5 +34,5 @@
   <xacro:create_link
       link_name="link3"
-      xyz_offset="-0.0679648513950829 -0.0125948841535013 0.0597190016437489"
+      xyz_offset="0 0 0"
       rpy_offset="0 0 0"
       mass="0.441881459418396"
@@ -41,5 +41,5 @@
   <xacro:create_link
       link_name="link4"
-      xyz_offset="-2.79564493776974E-08 -0.00496995620296214 0.0493158936775911"
+      xyz_offset="0 0 0"
       rpy_offset="0 0 0"
       mass="0.359995634810237"
@@ -48,6 +48,6 @@
   <xacro:create_link
       link_name="link5"
-      xyz_offset="-0.0043261798092078 0.0995606848099331 0.196143761355562"
-      rpy_offset="0 0 0"
+      xyz_offset="0 0 0"
+      rpy_offset="0 0 -0.187797428"
       mass="0.441881459418396"
       mesh_path="package://TechControlInterface/meshes"
@@ -55,5 +55,5 @@
   <xacro:create_link
       link_name="link6"
-      xyz_offset="0.000386879822536601 -0.0239742458499962 0.247370540938741"
+      xyz_offset="0 0 0"
       rpy_offset="0 0 0"
       mass="0.441881459418396"
@@ -68,5 +68,5 @@
   </joint>
   <!-- joints - main serial chain -->
-  <joint name="joint0" type="prismatic">
+  <joint name="joint0" type="fixed">
     <parent link="base_link"/>
     <child link="link0"/>
@@ -77,5 +77,5 @@
     <limit effort="1000.0" lower="-1" upper="1" velocity="2.5"/>
   </joint>
-  <joint name="joint1" type="prismatic">
+  <joint name="joint1" type="fixed">
     <parent link="link0"/>
     <child link="link1"/>
@@ -92,5 +92,5 @@
       xyz="0.149 -0.36401 0"
       rpy="1.680577537 0 1.5708" />
-    <axis xyz="1 0 0"/>
+    <axis xyz="-1 0 0"/>
     <limit effort="1000.0" lower="${-pi}" upper="${pi}" velocity="2.5"/>
   </joint>
@@ -118,14 +118,14 @@
     <origin
       xyz="0 -0.0735 0.0645"
-      rpy="1.5708 0.187869814 -3.1416" />
+      rpy="1.5708 0 -3.1416" />
     <axis xyz="0 0 -1"/>
     <limit effort="1000.0" lower="${-pi}" upper="${pi}" velocity="2.5"/>
   </joint>
-  <joint name="joint6" type="prismatic">
+  <joint name="joint6" type="fixed">
     <parent link="link5"/>
     <child link="link6"/>
     <origin
       xyz="0.0035379 0.14737 0.2235"
-      rpy="1.5708 0 -2.9537" />
+      rpy="1.5708 0 -3.141497428" />
     <axis xyz="0 0 1"/>
     <limit effort="1000.0" lower="-1" upper="1" velocity="2.5"/>

File: src/TechControlInterface/urdf/robot.urdf (robot description, URDF)
Before this commit: robot transport_robot, 8 links, 7 joints
Links:
- link base_link: geometry collision mesh filename=package://TechControlInterface/meshes/base_link.STL; visual mesh filename=package://TechControlInterface/meshes/base_link.STL
- link link0: geometry collision mesh filename=package://TechControlInterface/meshes/link0.STL; visual mesh filename=package://TechControlInterface/meshes/link0.STL
- link link1: geometry collision mesh filename=package://TechControlInterface/meshes/link1.STL; visual mesh filename=package://TechControlInterface/meshes/link1.STL
- link link2: geometry collision mesh filename=package://TechControlInterface/meshes/link2.STL; visual mesh filename=package://TechControlInterface/meshes/link2.STL
- link link3: geometry collision mesh filename=package://TechControlInterface/meshes/link3.STL; visual mesh filename=package://TechControlInterface/meshes/link3.STL
- link link4: geometry collision mesh filename=package://TechControlInterface/meshes/link4.STL; visual mesh filename=package://TechControlInterface/meshes/link4.STL
- link link5: geometry collision mesh filename=package://TechControlInterface/meshes/link5.STL; visual mesh filename=package://TechControlInterface/meshes/link5.STL
- link link6: geometry collision mesh filename=package://TechControlInterface/meshes/link6.STL; visual mesh filename=package://TechControlInterface/meshes/link6.STL
Joints:
- joint joint0: origin xyz=0 0 0 rpy=0 0 0 -> xyz=0 -1 0.061584 rpy=0 0 0
- joint joint2: origin xyz=0.149 -0.36401 0 rpy=0 0 1.5708 -> xyz=0.149 -0.36401 0 rpy=1.680577537 0 1.5708
- joint joint3: origin xyz=-0.01 0.027384 0.2485 rpy=0 0 0 -> xyz=-0.01 0.027384 0.2485 rpy=-0.317649924 0 0
- joint joint5: origin xyz=0 -0.0735 0.0645 rpy=1.5708 1.363 -3.1416 -> xyz=0 -0.0735 0.0645 rpy=1.5708 0.187869814 -3.1416

Commit message: UPDATE: add cartesian controller

File: src/TechControlInterface/description/ros2_control/TechJoints.ros2_control.xacro (robot description, xacro)
@@ -6,5 +6,12 @@
         <plugin>TechControlInterface/TechHardwareInterface</plugin>
         <param name="eth_device">${eth_device}</param>
+        <!-- <plugin>mock_components/GenericSystem</plugin> -->
       </hardware>
+      <!-- <joint name="${prefix}joint1">
+        <command_interface name="position"/>
+        <state_interface name="position"/>
+        <command_interface name="velocity"/>
+        <state_interface name="velocity"/>
+      </joint> -->
       <joint name="${prefix}joint2">
         <command_interface name="position"/>

Commit message: TMPSAVE

File: src/TechControlInterface/description/ros2_control/TechJoints.ros2_control.xacro (robot description, xacro)
@@ -1,47 +1,26 @@
 <?xml version="1.0"?>
 <robot xmlns:xacro="http://www.ros.org/wiki/xacro">
-  <xacro:macro name="TechJoints_ros2_control" params="name prefix eth_device">
+  <xacro:macro name="igh_ethercat_drive" params="name">
     <ros2_control name="${name}" type="system">
       <hardware>
-        <plugin>TechControlInterface/TechHardwareInterface</plugin>
-        <param name="eth_device">${eth_device}</param>
-        <!-- <plugin>mock_components/GenericSystem</plugin> -->
+        <plugin>ethercat_driver/EthercatDriver</plugin>
+        <param name="master_id">0</param>
+        <param name="control_frequency">1000</param>
       </hardware>
-      <!-- <joint name="${prefix}joint1">
+      <joint name="joint2">
+        <state_interface name="position"/>
+        <state_interface name="velocity"/>
+        <state_interface name="effort"/>
         <command_interface name="position"/>
-        <state_interface name="position"/>
         <command_interface name="velocity"/>
-        <state_interface name="velocity"/>
-      </joint> -->
-      <joint name="${prefix}joint2">
-        <command_interface name="position"/>
-        <state_interface name="position"/>
-        <command_interface name="velocity"/>
-        <state_interface name="velocity"/>
+        <command_interface name="reset_fault"/>
+        <ec_module name="Tech">
+          <plugin>ethercat_generic_plugins/EcCiA402Drive</plugin>
+          <param name="alias">0</param>
+          <param name="position">0</param>
+          <param name="mode_of_operation">8</param>
+          <param name="slave_config">$(find TechControlInterface)/drive_xml/tech_driver.yaml</param>
+        </ec_module>
       </joint>
-      <joint name="${prefix}joint3">
-        <command_interface name="position"/>
-        <state_interface name="position"/>
-        <command_interface name="velocity"/>
-        <state_interface name="velocity"/>
-      </joint>
-      <joint name="${prefix}joint4">
-        <command_interface name="position"/>
-        <state_interface name="position"/>
-        <command_interface name="velocity"/>
-        <state_interface name="velocity"/>
-      </joint>
-        <joint name="${prefix}joint5">
-        <command_interface name="position"/>
-        <state_interface name="position"/>
-        <command_interface name="velocity"/>
-        <state_interface name="velocity"/>
-      </joint>
-      <!-- <joint name="${prefix}joint6">
-        <command_interface name="position"/>
-        <state_interface name="position"/>
-        <command_interface name="velocity"/>
-        <state_interface name="velocity"/>
-      </joint> -->
     </ros2_control>
   </xacro:macro>

File: src/TechControlInterface/description/urdf/actuator.xacro (robot description, xacro)
@@ -8,4 +8,4 @@
   <link name="world"/>
   <xacro:TechRobot/>
-  <xacro:TechJoints_ros2_control name="TechJointsRos2Control" prefix="$(arg prefix)" eth_device="$(arg eth_device)" />
+  <xacro:igh_ethercat_drive name="igh_ethercat_drive" />
 </robot>
